File: RP2350_60QFN_minimal.kicad_pcb (KiCad board)
At the start: 2 copper layers, 14 x 54 mm, 38 parts, among them J1 Conn_01x02_Pin, J3 SM03B-SRSS-TB, J5 Bus Out, SW1 SW_Push, U1 W25Q128JVS, U2 LMR50410Y3FQDBVRQ1, U3 RP2350_60QFN, U4 MAX3078E, Y1 ABM8-272-T3

Commit message: All parts in stock
Connections:
- J1 pad : GND -> (no net)
