File: RP2350_60QFN_minimal.kicad_sch (KiCad schematic)
At the start: 38 parts, among them J1 Conn_01x02_Pin, J3 SM03B-SRSS-TB, J5 Bus Out, SW1 SW_Push, U1 W25Q128JVS, U2 LMR50410Y3FQDBVRQ1, U3 RP2350_60QFN, U4 MAX3078E, Y1 ABM8-272-T3

Commit message: All parts in stock
Parts:
- C1, C12, C13, C14, C15, C16, C17, C18, C19, C20, C4, C6, C9: LCSC PN C307419 -> (none); LCSC Part # (none) -> C307419
- C10, C11, C5, C7: LCSC PN C2932473 -> (none); LCSC Part # (none) -> C2932473
- C2, C3: LCSC PN C326803 -> (none); LCSC Part # (none) -> C326803
- C8: LCSC PN C76991 -> (none); LCSC Part # (none) -> C76991
- J1: LCSC PN C431092 -> (none); LCSC Part # (none) -> C431092
- J3: LCSC PN C160403 -> (none); LCSC Part # (none) -> C160403
- J5: LCSC PN C265068 -> (none); LCSC Part # (none) -> C265068
- L1, L2: LCSC PN C42411119 -> (none); LCSC Part # (none) -> C42411119
- R1: LCSC PN C190095 -> (none); LCSC Part # (none) -> C190095
- R2: LCSC PN C852624 -> (none); LCSC Part # (none) -> C852624
- R3, R4: LCSC PN C106235 -> (none); LCSC Part # (none) -> C106235
- R5: LCSC PN C138002 -> (none); LCSC Part # (none) -> C138002
- R6: LCSC PN C60490 -> (none); LCSC Part # (none) -> C60490
- R7: LCSC PN C114758 -> (none); LCSC Part # (none) -> C114758
- SW1: LCSC PN C18198078 -> (none); LCSC Part # (none) -> C22375314
- U1: LCSC PN C113767 -> (none); LCSC Part # (none) -> C113767
- U2: LCSC PN C5219374 -> (none); LCSC Part # (none) -> C5219374
- U3: LCSC PN C42411118 -> (none); LCSC Part # (none) -> C42411118
- U4: LCSC PN C42396723 -> (none); LCSC Part # (none) -> C2671519
- Y1: LCSC PN C20625731 -> (none); LCSC Part # (none) -> C20625731
Connections:
- net RUN: now also SW1.1; no longer SW1.2
- net at R4.1: now also SW1.2; no longer SW1.1
